Commit message: Fix camera orientation

File: src/abb_camera_simulation/urdf/abb_irb4600_60_205_macro.xacro (robot description, xacro)
@@ -185,5 +185,5 @@
         <link name="${prefix}tool0"/>
         <!-- end of link list -->
-        <link name="kinect_mesh">
+        <link name="${prefix}kinect_mesh">
             <visual>
                 <origin xyz="0 0 0" rpy="0 0 0" />
@@ -202,5 +202,5 @@
             </collision>
             <inertial>
-                <origin xyz="0 0 0" rpy="0 0 0"/>
+                <origin xyz="0 0 0" rpy="0 1.57 0"/>
                 <mass value="0.1"/>
                 <inertia
@@ -210,7 +210,7 @@
             </inertial>
         </link>
-        <link name="look_at"/>
+        <link name="${prefix}look_at"/>
         <joint name="${prefix}base_to_lookat" type="fixed">
-            <origin xyz="1 0 0" rpy="0 0 0" />
+            <origin xyz="1 0 0" rpy="0 1.57 0" />
             <parent link="${prefix}base_link"/>
             <child link="look_at"/>
@@ -265,8 +265,8 @@
             <origin xyz="0.135 0 0" rpy="0 1.570796 0"/>
         </joint>
-        <joint name="to_kinect" type="fixed">
+        <joint name="${prefix}to_kinect" type="fixed">
             <parent link="${prefix}tool0"/>
             <child link="kinect_frame"/>
-            <origin xyz="0 0 0.015" rpy="0 0 1.57"/>
+            <origin xyz="0 0 0.015" rpy="0.63 0.89 1.57"/>
             <!--
             Translation
@@ -285,5 +285,5 @@
   -2.17805"/>-->
         </joint>
-        <joint name="to_kinect_mesh" type="revolute">
+        <joint name="${prefix}to_kinect_mesh" type="revolute">
             <parent link="${prefix}tool0"/>
             <child link="kinect_mesh"/>
@@ -292,5 +292,5 @@
             <origin xyz="0 0 0.015" rpy="0 0 1.57"/>
         </joint>
-        <link name ="kinect_frame"/>
+        <link name ="${prefix}kinect_frame"/>
         <transmission name="tran1">
             <type>transmission_interface/SimpleTransmission</type>
