Commit message: Volumetric basic

File: src/abb_camera_simulation/urdf/abb_irb4600_60_205.urdf (robot description, URDF)
Before this commit: robot abb_irb4600_60_205, 8 links, 7 joints
Links:
- added link kinect; collision mesh filename=package://abb_camera_simulation/meshes/kinect/collision/kin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 scale=0.001 0.001 0.001; visual mesh filename=package://abb_camera_simulation/meshes/kinect/visual/kinect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 scale=0.001 0.001 0.001
Joints:
- added joint tool0-kinect: type fixed, parent tool0, child kinect, origin xyz=0.135 0 0 rpy=0 1.570796 0

File: src/abb_camera_simulation/urdf/abb_irb4600_60_205.xacro (robot description, xacro)
@@ -2,5 +2,5 @@
 <robot name="abb_irb" xmlns:xacro="http://ros.org/wiki/xacro">
     <xacro:include filename="$(find abb_camera_simulation)/urdf/abb_irb4600_60_205.gazebo" />
-  <!--  <xacro:include filename = "$/home/user/model_editor_models/abb_irb/model.sdf")/> -->
+  <!--<xacro:include filename = "$/home/user/model_editor_models/abb_irb/model.sdf")/>-->
 	<xacro:include filename="$(find abb_camera_simulation)/urdf/abb_irb4600_60_205_macro.xacro" />
 	<xacro:abb_irb4600_60_205 prefix=""/>

File: src/abb_camera_simulation/urdf/abb_irb4600_60_205_macro.xacro (robot description, xacro)
@@ -187,5 +187,5 @@
         <link name="${prefix}kinect_mesh">
             <visual>
-                <origin xyz="0 0 0" rpy="0 0 0" />
+                <origin xyz="0 0 0" rpy="0 1.57 0" />
                 <geometry>
                     <mesh filename="package://abb_camera_simulation/meshes/kinect/visual/kinect_sensor.stl" scale ="0.001 0.001 0.001"/>
@@ -196,5 +196,5 @@
             </visual>
             <collision>
-                <origin xyz="0 0 0" rpy="0 0 0" />
+                <origin xyz="0 0 0" rpy="0 1.57 0" />
                 <geometry>
                     <mesh filename="package://abb_camera_simulation/meshes/kinect/collision/kinect_sensor.stl" scale ="0.001 0.001 0.001"/>
@@ -202,5 +202,5 @@
             </collision>
             <inertial>
-                <origin xyz="0 0 0" rpy="0 1.57 0"/>
+                <origin xyz="0 0 0" rpy="0 0 0"/>
                 <mass value="0.1"/>
                 <inertia
@@ -268,20 +268,5 @@
             <parent link="${prefix}tool0"/>
             <child link="kinect_frame"/>
-            <origin xyz="0 0 0.015" rpy="0.63 0.89 1.57"/>
-            <!--
-            Translation
-            -0.0694681
-            -0.284737
-            0.247462
-            Rotation
-            -1.61514
-            -0.043724
-            -2.17802
-            <origin xyz="-0.0695877
- -0.285281
-  0.240969"
-                    rpy=" -1.61039
--0.0438775
-  -2.17805"/>-->
+            <origin xyz="0 0 0" rpy="0 0 0"/>
         </joint>
         <joint name="${prefix}to_kinect_mesh" type="revolute">

Commit message: Move planning

File: src/abb_camera_simulation/urdf/abb_irb4600_60_205.urdf (robot description, URDF)
Before this commit: robot abb_irb4600_60_205, 9 links, 8 joints
Links:
- removed link kinect
- link tool0: geometry collision mesh filename=package://abb_camera_simulation/meshes/kinect/collision/kin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 scale=0.001 0.001 0.001; visual mesh filename=package://abb_camera_simulation/meshes/kinect/visual/kinect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 scale=0.001 0.001 0.001
Joints:
- removed joint tool0-kinect
